Commit message: urdf

File: urdfs/mujocomodels/indy7.urdf (robot description, URDF)
Before this commit: robot indy, 10 links, 9 joints
Links:
- removed link end_effector
- link link0: geometry collision mesh filename=Indy7_0_c.stl; visual mesh filename=Indy7_0_v.stl
- link link1: geometry collision mesh filename=Indy7_1_c.stl; visual mesh filename=Indy7_1_v.stl
- link link2: geometry collision mesh filename=Indy7_2_c.stl; visual mesh filename=Indy7_2_v.stl
- link link3: geometry collision mesh filename=Indy7_3_c.stl; visual mesh filename=Indy7_3_v.stl
- link link4: geometry collision mesh filename=Indy7_4_c.stl; visual mesh filename=Indy7_4_v.stl
- link link5: geometry collision mesh filename=Indy7_5_c.stl; visual mesh filename=Indy7_5_v.stl
- link link6: geometry collision mesh filename=Indy7_6_c.stl; visual mesh filename=Indy7_6_v.stl
Joints:
- removed joint end_effector_joint
