Commit message: checkpoint

File: urdfs/indy7.urdf (robot description, URDF)
Before this commit: robot indy, 9 links, 8 joints
Links:
- link link0: geometry collision mesh filename=meshes/indy7/collision/Indy7_0.stl; visual mesh filename=meshes/indy7/visual/Indy7_0.stl
- link link1: geometry collision mesh filename=meshes/indy7/collision/Indy7_1.stl; visual mesh filename=meshes/indy7/visual/Indy7_1.stl
- link link2: geometry collision mesh filename=meshes/indy7/collision/Indy7_2.stl; visual mesh filename=meshes/indy7/visual/Indy7_2.stl
- link link3: geometry collision mesh filename=meshes/indy7/collision/Indy7_3.stl; visual mesh filename=meshes/indy7/visual/Indy7_3.stl
- link link4: geometry collision mesh filename=meshes/indy7/collision/Indy7_4.stl; visual mesh filename=meshes/indy7/visual/Indy7_4.stl
- link link5: geometry collision mesh filename=meshes/indy7/collision/Indy7_5.stl; visual mesh filename=meshes/indy7/visual/Indy7_5.stl
- link link6: geometry collision mesh filename=meshes/indy7/collision/Indy7_6.stl; visual mesh filename=meshes/indy7/visual/Indy7_6.stl

Commit message: benchmark

File: urdfs/indy7.urdf (robot description, URDF)
Before this commit: robot indy, 10 links, 9 joints
Joints:
- joint end_effector_joint: origin xyz=0 0 0.06 rpy=0 0 0 -> xyz=0 0 0.0 rpy=0 0 0

File: urdfs/indy7_limited.urdf (robot description, URDF)
Before this commit: robot indy, 10 links, 9 joints
Joints:
- joint tcp: origin xyz=0.0                          0.0                          0.06 rpy=0.0                         0.0                         0.0 -> xyz=0.0                          0.0                          0.0 rpy=0.0                         0.0                         0.0

File: urdfs/mujocomodels/indy7.urdf (robot description, URDF)
Before this commit: robot indy, 9 links, 8 joints
Joints:
- joint tcp: origin xyz=0.0                          0.0                          0.06 rpy=0.0                         0.0                         0.0 -> xyz=0.0                          0.0                          0.0 rpy=0.0                         0.0                         0.0
